File: IMU.kicad_sch (KiCad schematic)
At the start: 6 parts, among them U2 BMI323, U3 W25Q128JVSIQ

Commit message: Completed Schematic
Parts:
- removed U2: BMI323, BMI323_BOS, symbol BMI323:BMI323
- added C30: 100 nF, symbol Device:C_Small
- added R17: 10k, symbol Device:R_Small
- added R18: B57332V5103F360, B57332V5103F360:TRES_B57332V5103F360, symbol B57332V5103F360:B57332V5103F360
- added U6: BMI323, BMI323:BMI323_BOS, symbol BMI323:BMI323
- U3: footprint SOIC_128JVSIQ_WIN -> W25Q128JVSIQ:SOIC_128JVSIQ_WIN
Connections:
- net +3V3: now also R17.1, U6.5 (VDDIO), U6.8 (VDD)
- net GND: now also C30.2, R18.2, U6.6 (GNDIO), U6.7 (GND)
- net INT1: now also U6.4 (INT1)
- net INT2: now also U6.9 (INT2)
- net SPI2_MISO: now also U6.1 (SDO)
- net SPI2_MOSI: now also U6.14 (SDX)
- net SPI2_NSS: now also U6.12 (CSB)
- net SPI2_SCK: now also U6.13 (SCX)
- new net TEMP_SENSE_ADC: C30.1, R17.2, R18.1
Other:
- note added: "TEMP SENSE"

Commit message: PCB Layout Component placement progress
Parts:
- C13, C14, C15, C30: footprint (none) -> Capacitor_SMD:C_0603_1608Metric
- R17, R6: footprint (none) -> Resistor_SMD:R_0603_1608Metric
Changed lines of the file:
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@@
 			)
 		)
-		(property "Footprint" ""
+		(property "Footprint" "Capacitor_SMD:C_0603_1608Metric"
 			(at 26.67 118.11 0)
 			(hide yes)
@@
 			)
 		)
-		(property "Footprint" ""
+		(property "Footprint" "Resistor_SMD:R_0603_1608Metric"
 			(at 36.83 96.52 0)
 			(hide yes)
@@
 			)
 		)
-		(property "Footprint" ""
+		(property "Footprint" "Capacitor_SMD:C_0603_1608Metric"
 			(at 38.1 57.15 0)
 			(hide yes)
@@
 			)
 		)
-		(property "Footprint" ""
+		(property "Footprint" "Capacitor_SMD:C_0603_1608Metric"
 			(at 102.87 57.15 0)
 			(hide yes)
@@
 			)
 		)
-		(property "Footprint" ""
+		(property "Footprint" "Resistor_SMD:R_0603_1608Metric"
 			(at 154.94 34.29 0)
 			(hide yes)
@@
 			)
 		)
-		(property "Footprint" ""
+		(property "Footprint" "Capacitor_SMD:C_0603_1608Metric"
 			(at 254 55.88 0)
 			(hide yes)
